File: quadcopter.sch (EAGLE design)
At the start: 0 parts

Commit message: Quadcopter schematic done
Parts:
- added A: ANTENNA2SMD5, quadparts_prebuilt:ANTENNA2SMD5
- added B1: BALUN0805, quadparts_prebuilt:BALUN0805
- added BATT1: BATTERY, quadparts_prebuilt:BATTERY
- added C1: 22pF, quadparts_prebuilt:CAPACITOR-NP_SMD-2012-0805_CERAMIC-22PF
- added C10, C12, C14, C21, C22, C23, C24, C9: 0.1uF, quadparts_prebuilt:CAPACITOR-NP_SMD-2012-0805_CERAMIC-0.1UF
- added C11: 10uF, quadparts_prebuilt:CAPACITOR-NP_SMD-2012-0805_CERAMIC-10UF
- added C13: 0.01uF, quadparts_prebuilt:CAPACITOR-NP_SMD-2012-0805_CERAMIC-0.01UF
- added C15, C16, C5, C6, C7, C8: 1uF, quadparts_prebuilt:CAPACITOR-NP_SMD-2012-0805_CERAMIC-1UF
- added C17, C18, C19, C20: 220uF, quadparts_prebuilt:CAPACITOR-POL_SMD-7043-D_TANTALUM-220UF
- added C2: 0.75pF, quadparts_prebuilt:CAPACITOR-NP_SMD-2012-0805_CERAMIC-0.75PF
- added C3, C4: 12pF, quadparts_prebuilt:CAPACITOR-NP_SMD-2012-0805_CERAMIC-12PF
- added D1, D2, D3, D4: 360mV, quadparts_prebuilt:DIODE-SCHOTTKY_SMD-SOD123-360MV
- added D5: RED, custom:LED_RED
- added D6: GREEN, custom:LED_GREEN
- added D7: BLUE, custom:LED_BLUE
- added J1: AVR_SPI_PRG_6NS, quadparts_prebuilt:AVR_SPI_PRG_6NS
- added J2: (no value), custom:MALE_HEADER_2POS-2X1-0.1IN
- added J3: (no value), quadparts_prebuilt:SIP-10_TH-254X10
- added JP1: FTDI_BASICPTH, quadparts_prebuilt:FTDI_BASICPTH
- added M1, M2, M3, M4: MOTOR_PADS, quadparts_prebuilt:MOTOR_PADS
- added N1: NET_BRIDGE, custom:NET_BRIDGE
- added Q1, Q2, Q3, Q4: MOSFET_SOT-23, custom:MOSFET_SOT-23
- added R1, R11, R2, R3, R5, R7, R9: 10K, quadparts_prebuilt:RESISTOR_SMD-2012-0805-10K
- added R10, R12, R13, R14, R4, R6, R8: 100, quadparts_prebuilt:RESISTOR_SMD-2012-0805-100
- added REG: TPS73633-DBVT, quadparts_prebuilt:TPS73633-DBVT
- added SW1: PUSHBUTTON_SMD-VERTICAL-1, quadparts_prebuilt:PUSHBUTTON_SMD-VERTICAL-1
- added U1: ATMEGA128RFA1, quadparts_prebuilt:ATMEGA128RFA1
- added U2: IMU_LSM9DS1TR, custom:IMU_LSM9DS1TR
- added Y1: 16MHz, quadparts_prebuilt:CRYSTAL5X3
Connections:
- new net 3V: C10.1, C11.1, C12.1, C16.1, C7.1, C8.1, J3.2, R1.2, R2.2, R3.2, REG.OUT, U1.DEVDD, U1.EVDD, U2.CS_A/G, U2.CS_M, U2.DEN_A/G, U2.SDO_A/G, U2.SDO_M, U2.VDD, U2.VDDIO
- new net BAT_GND: BATT1.N, C15.2, C17.-, C18.-, C19.-, C20.-, D7.C, J3.10, N1.1, Q1.S, Q2.S, Q3.S, Q4.S
- new net GND: B1.GND@5, C1.1, C10.2, C11.2, C12.2, C13.2, C14.2, C16.2, C2.2, C21.2, C22.2, C23.2, C24.2, C3.2, C4.2, C5.2, C6.2, C7.2, C8.2, D5.C, D6.C, J1.6, J3.1, JP1.6, N1.2, R11.1, R5.1, R7.1, R9.1, REG.GND, SW1.2, U1.AVSS, U1.AVSS_RFN, U1.AVSS_RFP, U1.CLKI, U1.DVSS, U1.TST, U2.GND, U2.RES
- new net MISO: J1.1, U1.PB3(MISO/PDO/PCINT3)
- new net MOSI: J1.4, U1.PB2(MOSI/PDI/PCINT2)
- new net N$1: C6.1, U1.AVDD
- new net N$10: D2.A, M2.V-, Q2.D
- new net N$11: C22.1, Q2.G, R6.2, R7.2
- new net N$12: BATT1.P, J2.1
- new net N$13: D1.A, M1.V-, Q1.D
- new net N$14: D3.A, M3.V-, Q3.D
- new net N$15: C9.1, JP1.1
- new net N$16: D6.A, R13.1
- new net N$17: C21.1, Q1.G, R4.2, R5.2
- new net N$18: C13.1, U2.CAP
- new net N$19: C14.1, U2.C1
- new net N$2: C5.1, U1.DVDD
- new net N$20: C23.1, Q3.G, R8.2, R9.2
- new net N$21: D4.A, M4.V-, Q4.D
- new net N$22: D7.A, R14.1
- new net N$23: C24.1, Q4.G, R10.2, R11.2
- new net N$3: B1.OUT1, U1.RFP
- new net N$4: B1.OUT2, U1.RFN
- new net N$5: B1.GND@2, C1.2
- new net N$6: C4.1, U1.XTAL1, Y1.2
- new net N$7: A.SIGNAL, B1.IN, C2.1
- new net N$8: C3.1, U1.XTAL2, Y1.1
- new net N$9: D5.A, R12.1
- new net PB6: R12.2, U1.PB6(OC1B/PCINT6)
- new net PB7: R13.2, U1.PB7(OC0A/OC1C/PCINT7)
- new net PWM1: J3.5, R4.1, U1.PE3(OC3A/AIN1)
- new net PWM2: J3.6, R6.1, U1.PE4(OC3B/INT4)
- new net PWM3: J3.7, R8.1, U1.PE5(OC3C/INT5)
- new net PWM4: J3.8, R10.1, U1.PB5(OC1A/PCINT5)
- new net RESET: C9.2, J1.5, R1.1, SW1.1, U1.RSTN
- new net RXD0: JP1.3, U1.PE0(RXD0/PCINT8)
- new net SCK: J1.3, U1.PB1(SCK/PCINT1)
- new net SCL: J3.3, R3.1, U1.PD0(SCL/INT0), U2.SCL/SPC
- new net SDA: J3.4, R2.1, U1.PD1(SDA/INT1), U2.SDA/SDI/SDO
- new net TXD0: JP1.2, U1.PE1(TXD0)
- new net VBAT: C15.1, C17.+, C18.+, C19.+, C20.+, D1.C, D2.C, D3.C, D4.C, J2.2, J3.9, M1.V+, M2.V+, M3.V+, M4.V+, R14.2, REG.EN, REG.IN
Other:
- note added: "Debugging Header"
- note added: "IMU"
- note added: "LEDs"
- note added: "Microcontroller"
- note added: "Motor Drivers"
- note added: "Power Supply"
