File: quadcopter.brd (EAGLE design)
At the start: 138 x 138 mm, 66 parts, among them J1 AVR_SPI_PRG_6NS, M1 MOTOR_PADS, M2 MOTOR_PADS, M3 MOTOR_PADS, M4 MOTOR_PADS, SW1 PUSHBUTTON_SMD-VERTICAL-1, U1 ATMEGA128RFA1, U2 IMU_LSM9DS1TR, Y1 16MHz

Commit message: Redesign board dimension
Parts:
- moved B1 298.1 mm to (17.3, -1.40), turned to 180 degrees
- moved A 297.1 mm to (22.8, -1.40)
- moved C2 295.6 mm to (19.5, 1.70), turned to 90 degrees
- moved U2 283.2 mm to (0.00, 0.00)
- moved C1 267.4 mm to (17.3, 1.70), turned to 270 degrees
- moved U1 261.9 mm to (9.50, -0.90), turned to 180 degrees
- moved BATT1 166.1 mm to (-116.3, -35.3)
- moved C13 166.1 mm to (-103.6, -4.85)
- moved C14 166.1 mm to (-92.1, -1.04)
- moved C17 166.1 mm to (-127.7, -20.1)
- moved C21 166.1 mm to (-99.8, -1.04)
- moved C8 166.1 mm to (-103.6, 10.4)
- moved D1 166.1 mm to (-112.5, -9.93)
- moved D5 166.1 mm to (-96.0, -20.1)
- moved J1 166.1 mm to (-116.3, -49.3)
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Connections:
- net N$1 renamed C6
- net N$10 renamed M2
- net N$11 renamed C22
- net N$12 renamed BATT1
- net N$13 renamed M1
- net N$14 renamed M3
- net N$15 renamed C9
- net N$16 renamed D6
- net N$17 renamed C21
- net N$18 renamed C13
- net N$19 renamed C14
- net N$2 renamed C5
- net N$20 renamed C23
- net N$21 renamed M4
- net N$22 renamed D7
- net N$23 renamed C24
- net N$3 renamed RFP
- net N$4 renamed RFN
- net N$5 renamed C1
- net N$6 renamed C4
- net N$7 renamed C2
- net N$8 renamed C3
- net N$9 renamed D5
Other:
- outline, holes or cut-outs redrawn

Commit message: Placed some parts on the board
Parts:
- moved R14 234.2 mm to (104.9, -9.30)
- moved R13 221.5 mm to (98.6, -9.30)
- moved R12 208.7 mm to (92.1, -9.30)
- moved D7 207.9 mm to (105.1, -5.29)
- moved D2 204.6 mm to (64.3, 76.0)
- moved C24 202.8 mm to (56.7, -95.8)
- moved M2 202.6 mm to (55.2, 76.8)
- moved R11 202.1 mm to (72.2, -84.8)
- moved R6 201.3 mm to (55.3, 87.6)
- moved M4 197.3 mm to (61.3, -76.1)
- moved D6 189.0 mm to (98.8, -5.29)
- moved D5 188.9 mm to (92.3, -5.19)
- moved R10 188.0 mm to (62.2, -85.9)
- moved R7 187.4 mm to (65.6, 87.3)
- moved C22 185.6 mm to (49.8, 97.6)
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Connections:
- net PWM1: now also J3.6; no longer J3.5
- net PWM2: now also J3.5; no longer J3.6
- net PWM3: now also J3.4; no longer J3.7
- net PWM4: now also J3.3; no longer J3.8
- net SCL: now also J3.8; no longer J3.3
- net SDA: now also J3.7; no longer J3.4

Commit message: Board design continue
Parts:
- moved M1 62.6 mm to (-24.2, 23.5), turned to 45 degrees
- moved C17 58.9 mm to (-30.2, 30.2), turned to 135 degrees
- moved C4 1.84 mm to (11.8, -11.6)
- moved Y1 1.84 mm to (10.2, -8.31)
- moved C5 1.84 mm to (11.9, 8.70)
- moved C7 1.84 mm to (9.80, 8.70)
- moved C1 1.84 mm to (18.5, 3.10)
- moved C2 1.84 mm to (20.7, 3.10)
- moved C3 1.84 mm to (8.60, -11.6)
- moved C8 1.84 mm to (7.70, 8.70)
- moved A 1.84 mm to (24.0, 0.00)
- moved B1 1.84 mm to (18.5, 0.00)
- moved U1 1.84 mm to (10.7, 0.50)
- moved C6 1.84 mm to (14.6, -7.70)
- moved C9 1.84 mm to (5.60, 8.70)

Commit message: Finished board design
Parts:
- added V1, V10, V11, V12, V13, V14, V15, V16, V17, V18, V19, V2, V20, V21, V22, V23, V24, V25, V26, V27, V28, V29, V3, V30, V31, V32, V33, V4, V5, V6, V7, V8, V9: (no value), quadparts_prebuilt:VIA-0.254MM
- moved R14 122.1 mm to (-16.6, 2.50), turned to 90 degrees
- moved D7 121.7 mm to (-16.6, -2.00), turned to 270 degrees
- moved R13 103.4 mm to (-2.50, 12.3), turned to 270 degrees
- moved D6 103.3 mm to (-2.50, 15.1)
- moved C23 94.5 mm to (-16.7, -18.3), turned to 225 degrees
- moved R12 92.3 mm to (2.40, 12.3), turned to 270 degrees
- moved D5 92.2 mm to (2.40, 15.1), turned to 180 degrees
- moved C24 87.9 mm to (18.3, -16.7), turned to 315 degrees
- moved C21 87.4 mm to (-18.3, 16.7), turned to 135 degrees
- moved R11 86.6 mm to (16.7, -18.3), turned to 135 degrees
- moved R8 86.4 mm to (-15.0, -15.0), turned to 225 degrees
- moved C22 85.9 mm to (16.7, 18.3), turned to 45 degrees
- moved R10 85.2 mm to (15.0, -15.0), turned to 315 degrees
- moved R7 85.0 mm to (18.3, 16.7), turned to 225 degrees
- moved R6 83.0 mm to (15.0, 15.0), turned to 45 degrees
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Connections:
- net 3V: now also V1.P1, V2.P1, V3.P1, V32.P1, V4.P1
- net BAT_GND: now also V5.P1, V6.P1, V7.P1, V8.P1
- net GND: now also V13.P1, V14.P1, V15.P1, V16.P1, V17.P1, V18.P1, V19.P1, V20.P1, V21.P1, V22.P1, V23.P1, V24.P1, V25.P1, V26.P1, V27.P1, V28.P1, V29.P1, V30.P1, V31.P1, V33.P1
- net VBAT: now also V10.P1, V11.P1, V12.P1, V9.P1
Routing:
- net GND: track 0.00 -> 224.4 mm, vias 0 -> 2
- net RESET: track 0.00 -> 89.8 mm
- net PWM2: track 0.00 -> 71.8 mm, vias 0 -> 1
- net 3V: track 0.00 -> 61.3 mm, vias 0 -> 5
- net PWM1: track 0.00 -> 54.3 mm
- net SDA: track 0.00 -> 53.9 mm, vias 0 -> 2
- net VBAT: track 0.00 -> 52.1 mm
- net PWM3: track 0.00 -> 47.9 mm
- net SCL: track 0.00 -> 44.7 mm, vias 0 -> 3
- net RXD0: track 0.00 -> 38.5 mm
- net PWM4: track 0.00 -> 35.9 mm, vias 0 -> 1
- net TXD0: track 0.00 -> 35.4 mm, vias 0 -> 1
- net BAT_GND: track 0.00 -> 32.1 mm, vias 0 -> 4
- net MISO: track 0.00 -> 29.5 mm
- net MOSI: track 0.00 -> 25.2 mm, vias 0 -> 1
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- added copper zone on layer 15, net 3V
- added copper zone on layer 2, net BAT_GND
- added copper zone on layer 1, net GND
- added copper zone on layer 2, net GND
- added copper zone on layer 15, net VBAT

Commit message: Modified board design
Parts:
- removed V2, V4: (no value), quadparts_prebuilt:VIA-0.254MM
- added V34: (no value), quadparts_prebuilt:VIA-0.254MM
- moved D6 30.7 mm to (2.50, -15.2), turned to 180 degrees
- moved D5 30.7 mm to (-2.40, -15.2), turned to 0 degrees
- moved SW1 29.2 mm to (-0.10, 13.8), turned to 270 degrees
- moved R13 25.2 mm to (2.50, -12.4), turned to 90 degrees
- moved R12 25.2 mm to (-2.40, -12.4), turned to 90 degrees
- moved R2 4.10 mm to (-6.10, -10.2)
- moved R3 4.10 mm to (-8.20, -10.2)
- moved C2 1.18 mm to (20.9, 4.25)
- moved V26 1.00 mm to (22.7, 3.20)
- moved A 0.79 mm to (24.2, 0.75)
- moved V17 0.70 mm to (22.0, 6.50)
- moved V21 0.70 mm to (18.0, 6.50)
- moved V22 0.70 mm to (19.0, 6.50)
- moved V23 0.70 mm to (20.0, 6.50)
- moved V24 0.70 mm to (21.0, 6.50)
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Connections:
- net 3V: no longer V2.P1, V4.P1
- net GND: now also V34.P1
Routing:
- net RESET: track 89.8 -> 53.5 mm
- net GND: track 224.4 -> 196.2 mm, vias 2 -> 1
- net PWM2: track 71.8 -> 48.8 mm, vias 1 -> 2
- net RXD0: track 38.5 -> 58.5 mm
- net PWM1: track 54.3 -> 70.4 mm, vias 0 -> 1
- net 3V: track 61.3 -> 48.6 mm, vias 5 -> 6
- net SDA: track 53.9 -> 43.0 mm, vias 2 -> 3
- net MISO: track 29.5 -> 22.6 mm, vias 0 -> 1
- net PWM3: track 47.9 -> 41.4 mm
- net MOSI: track 25.2 -> 20.5 mm
- net PB7: track 16.1 -> 12.5 mm, vias 2 -> 0
- net TXD0: track 35.4 -> 31.9 mm
- net BAT_GND: track 32.1 -> 34.8 mm
- net SCL: track 44.7 -> 46.4 mm
- net PB6: track 13.4 -> 15.0 mm
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